File: lpc-mcu.sch (KiCad schematic (older format))
At the start: 0 parts

Commit message: started on lpc-mcu and ucb sheets
Parts:
- added IC?: LPC11U14FBD48, LQFP48, symbol LPC11U14FBD48
Connections:
- new net 3V3: IC?.44 (VDD), IC?.8 (VDD)
- new net GND: IC?.41 (VSS), IC?.5 (VSS)
- new net PIO0_1: IC?.4 (PIO0_1/CLKOUT/CT32B0_MAT2/USB_FTOGGLE)
- new net USB_DM: IC?.19 (USB_DM)
- new net USB_DP: IC?.20 (USB_DP)
- new net USB_VBUS: IC?.14 (PIO0_3/USB_VBUS)
- new net nRESET: IC?.3 (nRESET/PIO0_0)
- new net nUSB_CONNECT: IC?.22 (PIO0_6/nUSB_CONNECT/SCK0)
Changed lines of the file:
@@
 $Descr A4 11693 8268
 encoding utf-8
-Sheet 1 6
+Sheet 2 6
 Title ""
 Date "26 dec 2014"
@@
 Comment4 ""
 $EndDescr
+$Comp
+L LPC11U14FBD48 IC?
+U 1 1 549D53F4
+P 5250 4200
+F 0 "IC?" H 4500 6250 40  0000 L BNN
+F 1 "LPC11U14FBD48" H 4550 2200 40  0000 L BNN
+F 2 "LQFP48" H 5250 4200 30  0000 C CIN
+F 3 "~" H 5250 4200 60  0000 C CNN
+	1    5250 4200
+	1    0    0    -1
+$EndComp
+Text GLabel 4050 3500 0    60   Input ~ 0
+3V3
+Text GLabel 4050 3850 0    60   Input ~ 0
+3V3
+Text GLabel 4050 3600 0    60   Input ~ 0
+GND
+Text GLabel 4050 3950 0    60   Input ~ 0
+GND
+Text GLabel 4050 4250 0    60   Input ~ 0
+USB_DM
+Text GLabel 4050 4350 0    60   Input ~ 0
+USB_DP
+Text Label 6600 2200 0    60   ~ 0
+nRESET
+Text GLabel 7050 2500 2    60   Input ~ 0
+USB_VBUS
+Text Label 6600 2300 0    60   ~ 0
+PIO0_1
+Wire Wire Line
+	6600 2300 6250 2300
+Wire Wire Line
+	6250 2200 6600 2200
+Wire Wire Line
+	7050 2500 6250 2500
+Text GLabel 7050 2800 2    60   Input ~ 0
+nUSB_CONNECT
+Wire Wire Line
+	7050 2800 6250 2800
+Wire Wire Line
+	4050 3500 4350 3500
+Wire Wire Line
+	4350 3600 4050 3600
+Wire Wire Line
+	4050 3850 4350 3850
+Wire Wire Line
+	4350 3950 4050 3950
+Wire Wire Line
+	4050 4250 4350 4250
+Wire Wire Line
+	4350 4350 4050 4350
 $EndSCHEMATC
