File: pcb/nrf24l01p.sch (KiCad schematic (older format))
At the start: 1 part

Commit message: moved everything into follower's preferred project layout
Parts:
- removed P?: USB, symbol CONN_4
Other:
- note removed: "Micro-USB connectors have five pins, and implement nUSB_CONNECT somehow, but I guess we'll just be using four?"
Changed lines of the file:
@@
 LIBS:contrib
 LIBS:valves
+LIBS:arm-swd-header
 LIBS:lpc11u14fbd48
 LIBS:nRF24L01+
 LIBS:pp_ws2812b
-LIBS:arm-swd-header
 LIBS:modular-arm-usb-cache
 EELAYER 27 0
@@
 $Descr A4 11693 8268
 encoding utf-8
-Sheet 3 6
+Sheet 1 6
 Title ""
-Date "26 dec 2014"
+Date ""
 Rev ""
 Comp ""
@@
 Comment4 ""
 $EndDescr
-Text GLabel 3750 2600 0    60   Input ~ 0
-USB_VBUS
-Text GLabel 3750 2800 0    60   Input ~ 0
-nUSB_CONNECT
-Text GLabel 3750 3000 0    60   Input ~ 0
-USB_DM
-Text GLabel 3750 3200 0    60   Input ~ 0
-USB_DP
-Text GLabel 3750 3400 0    60   Input ~ 0
-GND
-$Comp
-L CONN_4 P?
-U 1 1 549D55CB
-P 5650 3000
-F 0 "P?" V 5600 3000 50  0000 C CNN
-F 1 "USB" V 5700 3000 50  0000 C CNN
-F 2 "" H 5650 3000 60  0000 C CNN
-F 3 "" H 5650 3000 60  0000 C CNN
-	1    5650 3000
-	1    0    0    -1
-$EndComp
-Text Notes 2550 2200 0    60   ~ 0
-Micro-USB connectors have five pins, and implement nUSB_CONNECT somehow, but I guess we'll just be using four?
 $EndSCHEMATC
