File: pcb/nrf24l01p.sch (KiCad schematic (older format))
At the start: 1 part, among them U3 NRF24L01+

Commit message: updated kicad to latest version and fixed things that didn't show up properly (text, nrf24l01+ part)
Parts:
- removed U3: NRF24L01+, MODULE, symbol NRF24L01+
- added U3: nRF24L01+, MODULE, symbol nRF24L01+
Changed lines of the file:
@@
 LIBS:pp_ws2812b
 LIBS:modular-arm-usb-cache
-EELAYER 27 0
+EELAYER 25 0
 EELAYER END
 $Descr A4 11693 8268
@@
 Comment4 ""
 $EndDescr
-$Comp
-L NRF24L01+ U3
-U 1 1 549D5C9C
-P 5250 3550
-F 0 "U3" H 5250 3250 50  0000 C CNN
-F 1 "NRF24L01+" H 5250 3850 50  0000 C CNN
-F 2 "MODULE" H 5250 3650 50  0001 C CNN
-F 3 "DOCUMENTATION" H 5250 3500 50  0001 C CNN
-	1    5250 3550
-	1    0    0    -1
-$EndComp
 Text GLabel 4300 3350 0    60   Input ~ 0
 GND
@@
 Wire Wire Line
 	4500 3500 4300 3500
+$Comp
+L nRF24L01+ U3
+U 1 1 54A763FB
+P 5250 3550
+F 0 "U3" H 5250 3250 50  0000 C CNN
+F 1 "nRF24L01+" H 5250 3850 50  0000 C CNN
+F 2 "MODULE" H 5250 3650 50  0001 C CNN
+F 3 "DOCUMENTATION" H 5250 3500 50  0001 C CNN
+	1    5250 3550
+	1    0    0    -1
+$EndComp
 $EndSCHEMATC
