File: pcb/charging.sch (KiCad schematic (older format))
At the start: 0 parts

Commit message: tied up some loose ends in power.sch
Other:
- note added: "One day we'll implement USB battery charging :)"
Changed lines of the file:
@@
 Comment4 ""
 $EndDescr
+Text Notes 4300 3550 0    60   ~ 0
+One day we'll implement USB battery charging :)
 $EndSCHEMATC
